File: Led-cube-driver/Led-cube-driver.kicad_sch (KiCad schematic)
At the start: 31 parts, among them J1 Diodes-input, J2 Vin, J3 Diodes-output, J4 Layers-input, J5 Layers-output, Q1 BC547, Q2 BC547, Q3 BC547, Q4 BC547, U1 74HC164, U2 74HC164

Commit message: newFiles
Changed lines of the file:
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@@
   )
   (symbol (lib_id "74xx:74HC164") (at 188.468 77.724 0) (unit 1)
-    (in_bom yes) (on_board yes) (fields_autoplaced)
+    (in_bom yes) (on_board yes)
     (property "Reference" "U1" (id 0) (at 190.4874 62.484 0)
       (effects (font (size 1.27 1.27)) (justify left))
@@
       (effects (font (size 1.27 1.27)) (justify left))
     )
-    (property "Footprint" "74hc164:74hc164DIP" (id 2) (at 211.328 85.344 0))
+    (property "Footprint" "74hc164:74hc164DIP" (id 2) (at 187.96 52.07 0))
     (property "Datasheet" "https://assets.nexperia.com/documents/data-sheet/74HC_HCT164.pdf" (id 3) (at 211.328 85.344 0)
       (effects (font (size 1.27 1.27)) hide)
